Commit message: Fix XML namespace URLs and update robot base link origin in URDF files
Co-authored-by: Copilot <copilot@github.com>

File: puzzlebot_nv_ws/src/puzzlebot_ros2/puzzlebot_description/urdf/puzzlebot.xacro (robot description, xacro)
@@ -1,5 +1,5 @@
 <?xml version="1.0"?>
-<robot xmlns:xacro="https://www.ros.org/wiki/xacro" name="puzzlebot">
-    <xacro:args name="prefix" default="" />
+<robot xmlns:xacro="http://www.ros.org/wiki/xacro" name="puzzlebot">
+    <xacro:arg name="prefix" default="" />
     <xacro:include filename="$(find puzzlebot_description)/urdf/puzzlebot.urdf.xacro"/>
     <xacro:include filename="$(find puzzlebot_description)/urdf/puzzlebot_control.xacro"/>

File: puzzlebot_nv_ws/src/puzzlebot_ros2/puzzlebot_description/urdf/puzzlebot_control.xacro (robot description, xacro)
@@ -1,4 +1,4 @@
 <?xml version="1.0"?>
-<robot xmlns:xacro="https://www.ros.org/wiki/xacro">
+<robot xmlns:xacro="http://www.ros.org/wiki/xacro">
     <xacro:macro name= "puzzlebot_control" params="prefix">
         <gazebo>
@@ -12,8 +12,8 @@
                 <wheel_radius>0.05</wheel_radius>
                 <topic>${prefix}cmd_vel</topic>
-                <tf_topic>diff_drive_tf</tf_topic>
+                <tf_topic>/model/puzzlebot/tf</tf_topic>
                 <odom_topic>${prefix}odom</odom_topic>
-                <frame_id>${prefix}odom</frame_id> <! -- Father frame for odometry -->
-                <child_frame_id>${prefix}base_footprint</child_frame_id> <! -- Child frame for odometry -->
+                <frame_id>${prefix}odom</frame_id> <!-- Father frame for odometry -->
+                <child_frame_id>${prefix}base_link</child_frame_id> <!-- Child frame for odometry -->
                 <odom_publisher_frequency>50</odom_publisher_frequency>
                 <max_angular_acceleration>1.8</max_angular_acceleration>

File: puzzlebot_nv_ws/src/puzzlebot_ros2/puzzlebot_description/urdf/robot_base.xacro (robot description, xacro)
@@ -4,7 +4,7 @@
     <link name="base_link">
       <visual>
-        <origin xyz="0 0 0" rpy="0 0 0" />
+        <origin xyz="0 0 0.04" rpy="0 0 0" />
         <geometry>
-          <mesh filename="$(find puzzlebot_description)/meshes/Puzzlebot_Jetson_Lidar_Edition_Base.stl"
+          <mesh filename="package://puzzlebot_description/meshes/Puzzlebot_Jetson_Lidar_Edition_Base.stl"
                 scale="${mesh_scale} ${mesh_scale} ${mesh_scale}" />
         </geometry>
