Commit message: Add robot base joint and update navigation parameters for improved mapping and simulation

File: puzzlebot_nv_ws/src/puzzlebot_ros2/puzzlebot_description/urdf/robot_base.xacro (robot description, xacro)
@@ -2,4 +2,10 @@
 <robot xmlns:xacro="http://www.ros.org/wiki/xacro">
   <xacro:macro name="robot_base" params="base_length:=0.24 base_width:=0.16 base_height:=0.06 base_mass:=1.5 mesh_scale:=0.001">
+    <link name="base_footprint"/>
+    <joint name="base_footprint_joint" type="fixed">
+      <parent link="base_footprint"/>
+      <child link="base_link"/>
+      <origin xyz="0 0 0" rpy="0 0 0"/>
+    </joint>
     <link name="base_link">
       <visual>
