Commit message: Update robot_base.xacro and wheels.xacro: adjust mesh_scale and origin positions for improved geometry alignment
Co-authored-by: Copilot <copilot@github.com>

File: puzzlebot_nv_ws/src/puzzlebot_ros2/puzzlebot_description/urdf/robot_base.xacro (robot description, xacro)
@@ -1,5 +1,5 @@
 <?xml version="1.0"?>
 <robot xmlns:xacro="http://www.ros.org/wiki/xacro">
-  <xacro:macro name="robot_base" params="base_length:=0.24 base_width:=0.16 base_height:=0.06 base_mass:=1.5 mesh_scale:=0.001">
+  <xacro:macro name="robot_base" params="base_length:=0.24 base_width:=0.16 base_height:=0.06 base_mass:=1.5 mesh_scale:=1.0">
     <link name="base_link">
       <visual>

File: puzzlebot_nv_ws/src/puzzlebot_ros2/puzzlebot_description/urdf/wheels.xacro (robot description, xacro)
@@ -56,5 +56,5 @@
     <link name="caster_link">
       <visual>
-        <origin xyz="-0.147 0.0 -0.043" rpy="0 0 0" />
+        <origin xyz="0 0 0" rpy="0 0 0" />
         <geometry>
           <mesh filename="package://puzzlebot_description/meshes/Puzzlebot_Caster_Wheel.stl"
@@ -66,5 +66,5 @@
       </visual>
       <collision>
-        <origin xyz="-0.147 0.0 -0.043" rpy="0 0 0" />
+        <origin xyz="0 0 0" rpy="0 0 0" />
         <geometry>
           <mesh filename="package://puzzlebot_description/meshes/Puzzlebot_Caster_Wheel.stl"

Commit message: Update URDF and launch files: adjust mesh_scale parameters for consistency and enable localization in nav2_core.launch.xml
Co-authored-by: Copilot <copilot@github.com>

File: puzzlebot_nv_ws/src/puzzlebot_ros2/puzzlebot_description/urdf/robot_base.xacro (robot description, xacro)
@@ -1,5 +1,5 @@
 <?xml version="1.0"?>
 <robot xmlns:xacro="http://www.ros.org/wiki/xacro">
-  <xacro:macro name="robot_base" params="base_length:=0.24 base_width:=0.16 base_height:=0.06 base_mass:=1.5 mesh_scale:=0.001">
+  <xacro:macro name="robot_base" params="base_length:=0.24 base_width:=0.16 base_height:=0.06 base_mass:=1.5 mesh_scale:=1">
     <link name="base_link">
       <visual>

File: puzzlebot_nv_ws/src/puzzlebot_ros2/puzzlebot_description/urdf/sensors.xacro (robot description, xacro)
@@ -1,5 +1,5 @@
 <?xml version="1.0"?>
 <robot xmlns:xacro="http://www.ros.org/wiki/xacro">
-  <xacro:macro name="puzzlebot_sensors" params="lidar_x:=0.0 lidar_z:=0.055 lidar_mass:=0.05 mesh_scale:=0.001">
+  <xacro:macro name="puzzlebot_sensors" params="lidar_x:=0.0 lidar_z:=0.055 lidar_mass:=0.05 mesh_scale:=1">
     <link name="lidar_base_link" />
     <joint name="lidar_base_joint" type="fixed">

File: puzzlebot_nv_ws/src/puzzlebot_ros2/puzzlebot_description/urdf/wheels.xacro (robot description, xacro)
@@ -1,5 +1,5 @@
 <?xml version="1.0"?>
 <robot xmlns:xacro="http://www.ros.org/wiki/xacro">
-  <xacro:macro name="puzzlebot_wheels" params="wheel_radius:=0.033 wheel_width:=0.012 wheel_separation:=0.16 wheel_drop:=0.03 wheel_mass:=0.08 caster_x:=-0.08 caster_radius:=0.015 caster_mass:=0.02 mesh_scale:=0.001">
+  <xacro:macro name="puzzlebot_wheels" params="wheel_radius:=0.033 wheel_width:=0.012 wheel_separation:=0.16 wheel_drop:=0.03 wheel_mass:=0.08 caster_x:=-0.08 caster_radius:=0.015 caster_mass:=0.02 mesh_scale:=1">
     <link name="left_wheel_link">
       <visual>
