Commit message: Refactor URDF files for Puzzlebot: update joint definitions, fix link origins, enhance sensor configurations, and added stl files for geometry
Co-authored-by: Copilot <copilot@github.com>

File: puzzlebot_nv_ws/src/puzzlebot_ros2/puzzlebot_description/urdf/puzzlebot.urdf.xacro (robot description, xacro)
@@ -5,4 +5,12 @@
   <xacro:include filename="$(find puzzlebot_description)/urdf/wheels.xacro" />
   <xacro:include filename="$(find puzzlebot_description)/urdf/sensors.xacro" />
+<!--<link name="base_footprint"/>-->
+  <!-- Fixed joint connecting base_footprint to base_link -->
+  <!-- base_footprint is at ground level, base_link is offset upward -->
+  <!-- <joint name="base_link_joint" type="fixed">
+    <parent link="base_footprint" />
+    <child link="base_link" />
+    <origin xyz="0.052 0 0.05"/>
+  </joint> -->
   <xacro:robot_base />
   <xacro:puzzlebot_wheels />

File: puzzlebot_nv_ws/src/puzzlebot_ros2/puzzlebot_description/urdf/puzzlebot_control.xacro (robot description, xacro)
@@ -16,5 +16,5 @@
                 <frame_id>${prefix}odom</frame_id> <!-- Father frame for odometry -->
                 <child_frame_id>${prefix}base_link</child_frame_id> <!-- Child frame for odometry -->
-                <odom_publisher_frequency>50</odom_publisher_frequency>
+                <odom_publish_frequency>50</odom_publish_frequency>
                 <max_angular_acceleration>1.8</max_angular_acceleration>
                 <max_angular_velocity>13.0</max_angular_velocity>

File: puzzlebot_nv_ws/src/puzzlebot_ros2/puzzlebot_description/urdf/robot_base.xacro (robot description, xacro)
@@ -4,5 +4,5 @@
     <link name="base_link">
       <visual>
-        <origin xyz="0 0 0.04" rpy="0 0 0" />
+        <origin xyz="0 0 0.052" rpy="0 0 0" />
         <geometry>
           <mesh filename="package://puzzlebot_description/meshes/Puzzlebot_Jetson_Lidar_Edition_Base.stl"
@@ -14,7 +14,8 @@
       </visual>
       <collision>
-        <origin xyz="0 0 0.02" rpy="0 0 0" />
+        <origin xyz="0 0 0.052" rpy="0 0 0" />
         <geometry>
-          <box size="${base_length} ${base_width} ${base_height}" />
+          <mesh filename="package://puzzlebot_description/meshes/Puzzlebot_Jetson_Lidar_Edition_Base.stl"
+                scale="${mesh_scale} ${mesh_scale} ${mesh_scale}" />
         </geometry>
       </collision>

File: puzzlebot_nv_ws/src/puzzlebot_ros2/puzzlebot_description/urdf/sensors.xacro (robot description, xacro)
@@ -1,10 +1,11 @@
 <?xml version="1.0"?>
 <robot xmlns:xacro="http://www.ros.org/wiki/xacro">
-  <xacro:macro name="puzzlebot_sensors" params="lidar_x:=0.06 lidar_z:=0.055 lidar_mass:=0.05">
+  <xacro:macro name="puzzlebot_sensors" params="lidar_x:=0.0 lidar_z:=0.055 lidar_mass:=0.05 mesh_scale:=1.0">
     <link name="lidar_link">
       <visual>
-        <origin xyz="0 0 0" rpy="0 0 0" />
+        <origin xyz="0 0 0.021" rpy="0 0 0" />
         <geometry>
-          <box size="0.05 0.05 0.03" />
+          <mesh filename="package://puzzlebot_description/meshes/RPLidar.stl"
+                scale="${mesh_scale} ${mesh_scale} ${mesh_scale}" />
         </geometry>
         <material name="white">
@@ -13,7 +14,8 @@
       </visual>
       <collision>
-        <origin xyz="0 0 0" rpy="0 0 0" />
+        <origin xyz="0 0 0.021" rpy="0 0 0" />
         <geometry>
-          <box size="0.05 0.05 0.03" />
+          <mesh filename="package://puzzlebot_description/meshes/RPLidar.stl"
+                scale="${mesh_scale} ${mesh_scale} ${mesh_scale}" />
         </geometry>
       </collision>
@@ -25,4 +27,24 @@
       <origin xyz="${lidar_x} 0 ${lidar_z}" rpy="0 0 0" />
     </joint>
+    <gazebo reference="lidar_link">
+      <sensor name="lidar_sensor" type="gpu_lidar">
+          <topic>scan</topic>
+          <gz_frame_id>lidar_link</gz_frame_id>
+          <update_rate>10</update_rate>
+          <ray>
+              <scan>
+                  <horizontal>
+                      <samples>360</samples>
+                      <min_angle>-3.14159</min_angle>
+                      <max_angle>3.14159</max_angle>
+                  </horizontal>
+              </scan>
+              <range>
+                  <min>0.15</min>
+                  <max>12.0</max>
+              </range>
+          </ray>
+      </sensor>
+    </gazebo>
   </xacro:macro>
 </robot>

File: puzzlebot_nv_ws/src/puzzlebot_ros2/puzzlebot_description/urdf/wheels.xacro (robot description, xacro)
@@ -1,10 +1,11 @@
 <?xml version="1.0"?>
 <robot xmlns:xacro="http://www.ros.org/wiki/xacro">
-  <xacro:macro name="puzzlebot_wheels" params="wheel_radius:=0.033 wheel_width:=0.012 wheel_separation:=0.16 wheel_drop:=0.03 wheel_mass:=0.08 caster_x:=-0.08 caster_radius:=0.015 caster_mass:=0.02">
+  <xacro:macro name="puzzlebot_wheels" params="wheel_radius:=0.033 wheel_width:=0.012 wheel_separation:=0.16 wheel_drop:=0.03 wheel_mass:=0.08 caster_x:=-0.08 caster_radius:=0.015 caster_mass:=0.02 mesh_scale:=1.0">
     <link name="left_wheel_link">
       <visual>
         <origin xyz="0 0 0" rpy="1.5708 0 0" />
         <geometry>
-          <cylinder radius="${wheel_radius}" length="${wheel_width}" />
+          <mesh filename="package://puzzlebot_description/meshes/Puzzlebot_Wheel.stl"
+                scale="${mesh_scale} ${mesh_scale} ${mesh_scale}" />
         </geometry>
         <material name="black">
@@ -15,5 +16,6 @@
         <origin xyz="0 0 0" rpy="1.5708 0 0" />
         <geometry>
-          <cylinder radius="${wheel_radius}" length="${wheel_width}" />
+          <mesh filename="package://puzzlebot_description/meshes/Puzzlebot_Wheel.stl"
+                scale="${mesh_scale} ${mesh_scale} ${mesh_scale}" />
         </geometry>
       </collision>
@@ -30,5 +32,6 @@
         <origin xyz="0 0 0" rpy="1.5708 0 0" />
         <geometry>
-          <cylinder radius="${wheel_radius}" length="${wheel_width}" />
+          <mesh filename="package://puzzlebot_description/meshes/Puzzlebot_Wheel.stl"
+                scale="${mesh_scale} ${mesh_scale} ${mesh_scale}" />
         </geometry>
         <material name="black">
@@ -39,5 +42,6 @@
         <origin xyz="0 0 0" rpy="1.5708 0 0" />
         <geometry>
-          <cylinder radius="${wheel_radius}" length="${wheel_width}" />
+          <mesh filename="package://puzzlebot_description/meshes/Puzzlebot_Wheel.stl"
+                scale="${mesh_scale} ${mesh_scale} ${mesh_scale}" />
         </geometry>
       </collision>
@@ -52,7 +56,8 @@
     <link name="caster_link">
       <visual>
-        <origin xyz="0 0 0" rpy="0 0 0" />
+        <origin xyz="-0.147 0.0 -0.043" rpy="0 0 0" />
         <geometry>
-          <sphere radius="${caster_radius}" />
+          <mesh filename="package://puzzlebot_description/meshes/Puzzlebot_Caster_Wheel.stl"
+                scale="${mesh_scale} ${mesh_scale} ${mesh_scale}" />
         </geometry>
         <material name="dark_gray">
@@ -61,7 +66,8 @@
       </visual>
       <collision>
-        <origin xyz="0 0 0" rpy="0 0 0" />
+        <origin xyz="-0.147 0.0 -0.043" rpy="0 0 0" />
         <geometry>
-          <sphere radius="${caster_radius}" />
+          <mesh filename="package://puzzlebot_description/meshes/Puzzlebot_Caster_Wheel.stl"
+                scale="${mesh_scale} ${mesh_scale} ${mesh_scale}" />
         </geometry>
       </collision>

Commit message: Refactor URDF files for Puzzlebot: update link and joint definitions, adjust mesh_scale for improved sensor and wheel configurations, and enhance lidar integration for better navigation.
Co-authored-by: Copilot <copilot@github.com>

File: puzzlebot_nv_ws/src/puzzlebot_ros2/puzzlebot_description/urdf/puzzlebot.urdf.xacro (robot description, xacro)
@@ -5,12 +5,10 @@
   <xacro:include filename="$(find puzzlebot_description)/urdf/wheels.xacro" />
   <xacro:include filename="$(find puzzlebot_description)/urdf/sensors.xacro" />
-<!--<link name="base_footprint"/>-->
-  <!-- Fixed joint connecting base_footprint to base_link -->
-  <!-- base_footprint is at ground level, base_link is offset upward -->
-  <!-- <joint name="base_link_joint" type="fixed">
+  <link name="base_footprint" />
+  <joint name="base_footprint_joint" type="fixed">
     <parent link="base_footprint" />
     <child link="base_link" />
-    <origin xyz="0.052 0 0.05"/>
-  </joint> -->
+    <origin xyz="0 0 0" rpy="0 0 0" />
+  </joint>
   <xacro:robot_base />
   <xacro:puzzlebot_wheels />

File: puzzlebot_nv_ws/src/puzzlebot_ros2/puzzlebot_description/urdf/puzzlebot_control.xacro (robot description, xacro)
@@ -15,5 +15,5 @@
                 <odom_topic>${prefix}odom</odom_topic>
                 <frame_id>${prefix}odom</frame_id> <!-- Father frame for odometry -->
-                <child_frame_id>${prefix}base_link</child_frame_id> <!-- Child frame for odometry -->
+                <child_frame_id>${prefix}base_footprint</child_frame_id> <!-- Child frame for odometry -->
                 <odom_publish_frequency>50</odom_publish_frequency>
                 <max_angular_acceleration>1.8</max_angular_acceleration>

File: puzzlebot_nv_ws/src/puzzlebot_ros2/puzzlebot_description/urdf/robot_base.xacro (robot description, xacro)
@@ -1,5 +1,5 @@
 <?xml version="1.0"?>
 <robot xmlns:xacro="http://www.ros.org/wiki/xacro">
-  <xacro:macro name="robot_base" params="base_length:=0.24 base_width:=0.16 base_height:=0.06 base_mass:=1.5 mesh_scale:=1.0">
+  <xacro:macro name="robot_base" params="base_length:=0.24 base_width:=0.16 base_height:=0.06 base_mass:=1.5 mesh_scale:=0.001">
     <link name="base_link">
       <visual>

File: puzzlebot_nv_ws/src/puzzlebot_ros2/puzzlebot_description/urdf/sensors.xacro (robot description, xacro)
@@ -1,5 +1,17 @@
 <?xml version="1.0"?>
 <robot xmlns:xacro="http://www.ros.org/wiki/xacro">
-  <xacro:macro name="puzzlebot_sensors" params="lidar_x:=0.0 lidar_z:=0.055 lidar_mass:=0.05 mesh_scale:=1.0">
+  <xacro:macro name="puzzlebot_sensors" params="lidar_x:=0.0 lidar_z:=0.055 lidar_mass:=0.05 mesh_scale:=0.001">
+    <link name="lidar_base_link" />
+    <joint name="lidar_base_joint" type="fixed">
+      <parent link="base_link" />
+      <child link="lidar_base_link" />
+      <origin xyz="${lidar_x} 0 ${lidar_z}" rpy="0 0 0" />
+    </joint>
+    <link name="laser_frame" />
+    <joint name="laser_frame_joint" type="fixed">
+      <parent link="lidar_base_link" />
+      <child link="laser_frame" />
+      <origin xyz="0 0 0.021" rpy="0 0 0" />
+    </joint>
     <link name="lidar_link">
       <visual>
@@ -23,12 +35,12 @@
     </link>
     <joint name="lidar_joint" type="fixed">
-      <parent link="base_link" />
+      <parent link="laser_frame" />
       <child link="lidar_link" />
-      <origin xyz="${lidar_x} 0 ${lidar_z}" rpy="0 0 0" />
+      <origin xyz="0 0 0" rpy="0 0 0" />
     </joint>
     <gazebo reference="lidar_link">
       <sensor name="lidar_sensor" type="gpu_lidar">
           <topic>scan</topic>
-          <gz_frame_id>lidar_link</gz_frame_id>
+          <gz_frame_id>laser_frame</gz_frame_id>
           <update_rate>10</update_rate>
           <ray>

File: puzzlebot_nv_ws/src/puzzlebot_ros2/puzzlebot_description/urdf/wheels.xacro (robot description, xacro)
@@ -1,5 +1,5 @@
 <?xml version="1.0"?>
 <robot xmlns:xacro="http://www.ros.org/wiki/xacro">
-  <xacro:macro name="puzzlebot_wheels" params="wheel_radius:=0.033 wheel_width:=0.012 wheel_separation:=0.16 wheel_drop:=0.03 wheel_mass:=0.08 caster_x:=-0.08 caster_radius:=0.015 caster_mass:=0.02 mesh_scale:=1.0">
+  <xacro:macro name="puzzlebot_wheels" params="wheel_radius:=0.033 wheel_width:=0.012 wheel_separation:=0.16 wheel_drop:=0.03 wheel_mass:=0.08 caster_x:=-0.08 caster_radius:=0.015 caster_mass:=0.02 mesh_scale:=0.001">
     <link name="left_wheel_link">
       <visual>
