Commit message: Fix xacro include syntax and update launch file paths for consistency

File: puzzlebot_nv_ws/src/puzzlebot_ros2/puzzlebot_description/urdf/puzzlebot.urdf.xacro (robot description, xacro)
@@ -1,8 +1,8 @@
 <?xml version="1.0"?>
 <robot name="puzzlebot" xmlns:xacro="http://www.ros.org/wiki/xacro">
-  <xacro:include filename="$(find-pkg-share puzzlebot_description)/urdf/macros.xacro" />
-  <xacro:include filename="$(find-pkg-share puzzlebot_description)/urdf/robot_base.xacro" />
-  <xacro:include filename="$(find-pkg-share puzzlebot_description)/urdf/wheels.xacro" />
-  <xacro:include filename="$(find-pkg-share puzzlebot_description)/urdf/sensors.xacro" />
+  <xacro:include filename="$(find puzzlebot_description)/urdf/macros.xacro" />
+  <xacro:include filename="$(find puzzlebot_description)/urdf/robot_base.xacro" />
+  <xacro:include filename="$(find puzzlebot_description)/urdf/wheels.xacro" />
+  <xacro:include filename="$(find puzzlebot_description)/urdf/sensors.xacro" />
   <xacro:robot_base />
   <xacro:puzzlebot_wheels />

File: puzzlebot_nv_ws/src/puzzlebot_ros2/puzzlebot_description/urdf/robot_base.xacro (robot description, xacro)
@@ -6,5 +6,6 @@
         <origin xyz="0 0 0" rpy="0 0 0" />
         <geometry>
-          <mesh filename="package://puzzlebot_description/meshes/Puzzlebot_Jetson_Lidar_Edition_Base.stl" scale="${mesh_scale} ${mesh_scale} ${mesh_scale}" />
+          <mesh filename="$(find puzzlebot_description)/meshes/Puzzlebot_Jetson_Lidar_Edition_Base.stl"
+                scale="${mesh_scale} ${mesh_scale} ${mesh_scale}" />
         </geometry>
         <material name="gray">

Commit message: Fix - update mesh file paths to use package URI format and adjust transform_tolerance and initial pose settings in navigation parameters

File: puzzlebot_nv_ws/src/puzzlebot_ros2/puzzlebot_description/urdf/puzzlebot.urdf.xacro (robot description, xacro)
@@ -18,5 +18,5 @@
       <origin xyz="0 0.052 0" rpy="0 0 0" />
       <geometry>
-        <mesh filename="file://$(find puzzlebot_description)/meshes/Puzzlebot_Jetson_Lidar_Edition_Base.stl" scale="1 1 1"/>
+        <mesh filename="package://puzzlebot_description/meshes/Puzzlebot_Jetson_Lidar_Edition_Base.stl" scale="1 1 1"/>
       </geometry>
       <material name="red" />
@@ -25,5 +25,5 @@
       <origin xyz="0 0.052 0" rpy="0 0 0" />
       <geometry>
-        <mesh filename="file://$(find puzzlebot_description)/meshes/Puzzlebot_Jetson_Lidar_Edition_Base.stl" scale="1 1 1"/>
+        <mesh filename="package://puzzlebot_description/meshes/Puzzlebot_Jetson_Lidar_Edition_Base.stl" scale="1 1 1"/>
       </geometry>
     </collision>
@@ -46,5 +46,5 @@
       <origin xyz="0 0 0" rpy="-1.5708 0 0" />
       <geometry>
-        <mesh filename="file://$(find puzzlebot_description)/meshes/Puzzlebot_Wheel.stl" scale="1 1 1"/>
+        <mesh filename="package://puzzlebot_description/meshes/Puzzlebot_Wheel.stl" scale="1 1 1"/>
       </geometry>
       <material name="red" />
@@ -53,5 +53,5 @@
       <origin xyz="0 0 0" rpy="-1.5708 0 0" />
       <geometry>
-        <mesh filename="file://$(find puzzlebot_description)/meshes/Puzzlebot_Wheel.stl" scale="1 1 1"/>
+        <mesh filename="package://puzzlebot_description/meshes/Puzzlebot_Wheel.stl" scale="1 1 1"/>
       </geometry>
     </collision>
@@ -77,5 +77,5 @@
       <origin xyz="0 0 0" rpy="1.5708 0 0" />
       <geometry>
-        <mesh filename="file://$(find puzzlebot_description)/meshes/Puzzlebot_Wheel.stl" scale="1 1 1"/>
+        <mesh filename="package://puzzlebot_description/meshes/Puzzlebot_Wheel.stl" scale="1 1 1"/>
       </geometry>
       <material name="red" />
@@ -84,5 +84,5 @@
       <origin xyz="0 0 0" rpy="1.5708 0 0" />
       <geometry>
-        <mesh filename="file://$(find puzzlebot_description)/meshes/Puzzlebot_Wheel.stl" scale="1 1 1"/>
+        <mesh filename="package://puzzlebot_description/meshes/Puzzlebot_Wheel.stl" scale="1 1 1"/>
       </geometry>
     </collision>
@@ -107,5 +107,5 @@
     <visual>
       <geometry>
-        <mesh filename="file://$(find puzzlebot_description)/meshes/Puzzlebot_Caster_Wheel.stl" scale="1 1 1"/>
+        <mesh filename="package://puzzlebot_description/meshes/Puzzlebot_Caster_Wheel.stl" scale="1 1 1"/>
       </geometry>
       <material name="red" />
@@ -113,5 +113,5 @@
     <collision>
       <geometry>
-        <mesh filename="file://$(find puzzlebot_description)/meshes/Puzzlebot_Caster_Wheel.stl" scale="1 1 1"/>
+        <mesh filename="package://puzzlebot_description/meshes/Puzzlebot_Caster_Wheel.stl" scale="1 1 1"/>
       </geometry>
     </collision>

File: puzzlebot_nv_ws/src/puzzlebot_ros2/puzzlebot_description/urdf/sensors.xacro (robot description, xacro)
@@ -6,5 +6,5 @@
     frame_name:='laser_frame'
     parent:='base_link'
-    mesh_file:='file://$(find puzzlebot_description)/meshes/RPLidar.stl'
+    mesh_file:='package://puzzlebot_description/meshes/RPLidar.stl'
     lidar_base_mass:='0.1755'
     lidar_base_length:='0.08'

Commit message: Fix - cost scaling factor

File: puzzlebot_nv_ws/src/puzzlebot_ros2/puzzlebot_description/urdf/puzzlebot.urdf.xacro (robot description, xacro)
@@ -8,4 +8,5 @@
   <material name="red"><color rgba="1.0 0.0 0.0 1.0" /></material>
   <material name="yellow"><color rgba="1.0 1.0 0.0 1.0" /></material>
+  <material name="grey"><color rgba="0.5 0.5 0.5 1.0" /></material>
   <link name="base_footprint" />
   <!-- Base -->

Commit message: Fix - URDF component placement

File: puzzlebot_nv_ws/src/puzzlebot_ros2/puzzlebot_description/urdf/puzzlebot.urdf.xacro (robot description, xacro)
@@ -17,5 +17,5 @@
     </inertial>
     <visual>
-      <origin xyz="0 0.052 0" rpy="0 0 0" />
+      <origin xyz="0 0 0" rpy="0 0 0" />
       <geometry>
         <mesh filename="package://puzzlebot_description/meshes/Puzzlebot_Jetson_Lidar_Edition_Base.stl" scale="1 1 1"/>
@@ -24,5 +24,5 @@
     </visual>
     <collision>
-      <origin xyz="0 0.052 0" rpy="0 0 0" />
+      <origin xyz="0 0 0" rpy="0 0 0" />
       <geometry>
         <mesh filename="package://puzzlebot_description/meshes/Puzzlebot_Jetson_Lidar_Edition_Base.stl" scale="1 1 1"/>
@@ -33,5 +33,5 @@
     <parent link="base_footprint" />
     <child link="base_link" />
-    <origin xyz="0.052 0 0.05" />
+    <origin xyz="0 0 0.05" />
   </joint>
   <gazebo reference="base_link">
@@ -61,5 +61,5 @@
     <parent link="base_link" />
     <child link="right_wheel_link" />
-    <origin xyz="0 -0.095 -0.0025"/>
+    <origin xyz="0.025 -0.095 -0.0025"/>
     <axis xyz="0 1 0" />
   </joint>
@@ -92,5 +92,5 @@
     <parent link="base_link" />
     <child link="left_wheel_link" />
-    <origin xyz="0 0.095 -0.0025"/>
+    <origin xyz="0.025 0.095 -0.0025"/>
     <axis xyz="0 1 0" />
   </joint>
@@ -121,5 +121,5 @@
     <parent link="base_link" />
     <child link="caster_link" />
-    <origin xyz="-0.147 0 -0.043"/>
+    <origin xyz="-0.110 0 -0.043"/>
   </joint>
   <gazebo reference="caster_link">
@@ -129,4 +129,4 @@
   </gazebo>
   <xacro:puzzlebot_control prefix="$(arg prefix)" />
-  <xacro:puzzlebot_sensors prefix="$(arg prefix)" />
+  <xacro:puzzlebot_sensors prefix="$(arg prefix)" lidar_base_pos_x="0.06" />
 </robot>
