Commit message: Refactor lidar sensor configuration: rename links and joints for clarity and consistency
Co-authored-by: Copilot <copilot@github.com>

File: puzzlebot_nv_ws/src/puzzlebot_ros2/puzzlebot_description/urdf/sensors.xacro (robot description, xacro)
@@ -8,11 +8,5 @@
       <origin xyz="${lidar_x} 0 ${lidar_z}" rpy="0 0 0" />
     </joint>
-    <link name="laser_frame" />
-    <joint name="laser_frame_joint" type="fixed">
-      <parent link="lidar_base_link" />
-      <child link="laser_frame" />
-      <origin xyz="0 0 0.021" rpy="0 0 0" />
-    </joint>
-    <link name="lidar_link">
+    <link name="laser_frame">
       <visual>
         <origin xyz="0 0 0.021" rpy="0 0 0" />
@@ -34,10 +28,10 @@
       <xacro:box_inertial mass="${lidar_mass}" x="0.05" y="0.05" z="0.03" />
     </link>
-    <joint name="lidar_joint" type="fixed">
-      <parent link="laser_frame" />
-      <child link="lidar_link" />
-      <origin xyz="0 0 0" rpy="0 0 0" />
+    <joint name="laser_frame_joint" type="fixed">
+      <parent link="lidar_base_link" />
+      <child link="laser_frame" />
+      <origin xyz="0 0 0.021" rpy="0 0 0" />
     </joint>
-    <gazebo reference="lidar_link">
+    <gazebo reference="laser_frame">
       <sensor name="lidar_sensor" type="gpu_lidar">
           <topic>scan</topic>
