Commit message: cambios hechos con el profe

File: puzzlebot_nv_ws/src/puzzlebot_ros2/puzzlebot_description/urdf/sensors.xacro (robot description, xacro)
@@ -54,3 +54,137 @@
     </gazebo>
   </xacro:macro>
+  <!-- New macro added -->
+  <xacro:property name="M_PI" value="3.1415926535897931" />
+  <xacro:macro name="rpi_lidar_sensor" params="
+    prefix:=''
+    frame_name:='laser_frame'
+    parent:='base_link'
+    mesh_file:='file://$(find puzzlebot_description)/meshes/sensors/RPLidar.stl'
+    lidar_base_mass:='0.1755'
+    lidar_base_length:='0.08'
+    lidar_base_width:='0.07'
+    lidar_base_height:='0.05'
+    lidar_base_inertia_pos_x:='0.0'
+    lidar_base_inertia_pos_y:='0.0'
+    lidar_base_inertia_pos_z:='0.021'
+    lidar_base_inertia_pos_r:='0.0'
+    lidar_base_inertia_pos_p:='0.0'
+    lidar_base_inertia_pos_w:='0.0'
+    lidar_base_collision_pos_x:='0.0'
+    lidar_base_collision_pos_y:='0.0'
+    lidar_base_collision_pos_z:='0.021'
+    lidar_base_collision_pos_r:='0.0'
+    lidar_base_collision_pos_p:='0.0'
+    lidar_base_collision_pos_w:='0.0'
+    lidar_base_mesh_pos_x:='0.0'
+    lidar_base_mesh_pos_y:='0.0'
+    lidar_base_mesh_pos_z:='0.025'
+    lidar_base_mesh_pos_r:='0.0'
+    lidar_base_mesh_pos_p:='0.0'
+    lidar_base_mesh_pos_w:='0.0'
+    lidar_base_pos_x:='0.0'
+    lidar_base_pos_y:='0.00'
+    lidar_base_pos_z:='0.070'
+    lidar_base_pos_r:='0.0'
+    lidar_base_pos_p:='0.0'
+    lidar_base_pos_w:='0.0'
+    lidar_pos_x:='0.0'
+    lidar_pos_y:='0.00'
+    lidar_pos_z:='0.035'
+    lidar_pos_r:='0.0'
+    lidar_pos_p:='0.0'
+    lidar_pos_w:='0.0'
+    update_rate:='10'
+    ray_count:='360'
+    min_angle:='-3.14159'
+    max_angle:='3.14159'
+    min_range:='0.15'
+    max_range:='12.0'
+    range_resolution:='0.017'
+    topic_name:='scan'
+    always_on:='true'
+    visualize:='false'
+    ">
+    <link name="${prefix}lidar_base_link">
+        <visual>
+            <origin xyz="${lidar_base_mesh_pos_x} ${lidar_base_mesh_pos_y} ${lidar_base_mesh_pos_z}" rpy="${lidar_base_mesh_pos_r} ${lidar_base_mesh_pos_p} ${lidar_base_mesh_pos_w}"/>
+            <geometry>
+                <mesh filename="${mesh_file}"/>
+            </geometry>
+            <material name="grey"/>
+        </visual>
+        <collision>
+            <origin xyz="${lidar_base_collision_pos_x} ${lidar_base_collision_pos_y} ${lidar_base_collision_pos_z}" rpy="${lidar_base_collision_pos_r} ${lidar_base_collision_pos_p} ${lidar_base_collision_pos_w}"/>
+            <geometry>
+                <box size="${lidar_base_length} ${lidar_base_width} ${lidar_base_height}"/>
+            </geometry>
+        </collision>
+        <inertial>
+            <origin xyz="${lidar_base_inertia_pos_x} ${lidar_base_inertia_pos_y} ${lidar_base_inertia_pos_z}" rpy="${lidar_base_inertia_pos_r} ${lidar_base_inertia_pos_p} ${lidar_base_inertia_pos_w}"/>
+            <mass value="${lidar_base_mass}"/>
+            <xacro:box_inertia mass="${lidar_base_mass}" x="${lidar_base_length}" y="${lidar_base_width}" z="${lidar_base_height}" />
+        </inertial>
+    </link>
+    <link name="${prefix}laser_frame">
+        <visual>
+            <origin xyz="0 0 0" rpy="0 0 0"/>
+            <geometry>
+                <box size="0.005 0.005 0.005"/> <!-- Box shape for lidar -->
+            </geometry>
+            <material name="grey"/>
+        </visual>
+        <collision>
+            <origin xyz="0 0 0" rpy="0 0 0"/>
+            <geometry>
+                <box size="0.005 0.005 0.005"/>
+            </geometry>
+        </collision>
+        <inertial>
+            <origin xyz="0 0 0" rpy="0 0 0"/>
+            <mass value="1e-5"/>
+            <xacro:box_inertia mass="1e-5" x="0.005" y="0.005" z="0.005" />
+        </inertial>
+    </link>
+    <joint name="${prefix}lidar_base_joint" type="fixed">
+        <parent link="${prefix}${parent}"/>
+        <child link="${prefix}lidar_base_link"/>
+        <origin xyz="${lidar_base_pos_x} ${lidar_base_pos_y} ${lidar_base_pos_z}" rpy="${lidar_base_pos_r} ${lidar_base_pos_p} ${lidar_base_pos_w}"/>
+    </joint>
+    <joint name="${prefix}lidar_joint" type="fixed">
+        <parent link="${prefix}lidar_base_link"/>
+        <child link="${prefix}laser_frame"/>
+        <origin xyz="${lidar_pos_x} ${lidar_pos_y} ${lidar_pos_z}" rpy="${lidar_pos_r} ${lidar_pos_p} ${lidar_pos_w}"/>
+    </joint>
+    <gazebo reference="${prefix}laser_frame">
+        <sensor name="${prefix}lidar_sensor" type="gpu_lidar">
+            <topic>${prefix}${topic_name}</topic>
+            <gz_frame_id>${prefix}laser_frame</gz_frame_id>
+            <pose> 0 0 0 0 0 0 </pose>
+            <update_rate>${update_rate}</update_rate>
+            <always_on>${always_on}</always_on>
+            <visualize>${visualize}</visualize>
+            <ray>
+            <scan>
+                <horizontal>
+                <samples>${ray_count}</samples>
+                <resolution>1</resolution>
+                <min_angle>${min_angle}</min_angle>
+                <max_angle>${max_angle}</max_angle>
+                </horizontal>
+                <vertical>
+                <samples>1</samples>
+                <resolution>0.01</resolution>
+                <min_angle>0</min_angle>
+                <max_angle>0</max_angle>
+                </vertical>
+            </scan>
+            <range>
+                <min>${min_range}</min>
+                <max>${max_range}</max>
+                <resolution>${range_resolution}</resolution>
+            </range>
+            </ray>
+        </sensor>
+    </gazebo>
+  </xacro:macro>
 </robot>

Commit message: Add hardware bringup and navigation support for Puzzlebot Real Robot
- Introduced TROUBLESHOOTING.md for comprehensive debugging guidance on hardware issues.
- Created nav2_params_real.yaml for configuring navigation parameters specific to the real robot.
- Added slam_toolbox_real.yaml for SLAM configuration tailored to the physical robot.
- Implemented real_robot_core.launch.xml to start all necessary hardware drivers and publish the TF tree.
- Developed real_robot_nav2.launch.xml for running the Nav2 stack for autonomous navigation.
- Created real_robot_slam.launch.xml for generating maps using SLAM Toolbox.
- Added package.xml to define the package and its dependencies.
- Implemented puzzlebot_joint_state_publisher.py to publish joint states and odometry transforms.
- Developed puzzlebot_localization.py for odometry calculations based on encoder data.

File: puzzlebot_nv_ws/src/puzzlebot_ros2/puzzlebot_description/urdf/sensors.xacro (robot description, xacro)
@@ -1,5 +1,15 @@
 <?xml version="1.0"?>
 <robot xmlns:xacro="http://www.ros.org/wiki/xacro">
-  <xacro:macro name="puzzlebot_sensors" params="lidar_x:=0.0 lidar_z:=0.055 lidar_mass:=0.05 mesh_scale:=1">
+  <!--
+    puzzlebot_sensors — LiDAR mount and laser_frame definition.
+    Defines the physical TF chain:
+      base_link -> lidar_base_link -> laser_frame
+    The <gazebo> block below is SIMULATION ONLY — it configures the
+    gpu_lidar sensor plugin for Gazebo. On the real robot this block
+    is ignored; the RPLidar A1 driver (rplidar_ros) publishes /scan
+    directly to the laser_frame defined by the joints above.
+  -->
+  <xacro:macro name="puzzlebot_sensors"
+               params="lidar_x:=0.0 lidar_z:=0.055 lidar_mass:=0.05 mesh_scale:=1">
     <link name="lidar_base_link" />
     <joint name="lidar_base_joint" type="fixed">
@@ -33,158 +43,26 @@
       <origin xyz="0 0 0.021" rpy="0 0 0" />
     </joint>
+    <!-- SIMULATION ONLY — Gazebo gpu_lidar sensor plugin.
+         Not loaded when robot_state_publisher uses puzzlebot.urdf.xacro directly. -->
     <gazebo reference="laser_frame">
       <sensor name="lidar_sensor" type="gpu_lidar">
-          <topic>scan</topic>
-          <gz_frame_id>laser_frame</gz_frame_id>
-          <update_rate>10</update_rate>
-          <ray>
-              <scan>
-                  <horizontal>
-                      <samples>360</samples>
-                      <min_angle>-3.14159</min_angle>
-                      <max_angle>3.14159</max_angle>
-                  </horizontal>
-              </scan>
-              <range>
-                  <min>0.15</min>
-                  <max>12.0</max>
-              </range>
-          </ray>
+        <topic>scan</topic>
+        <gz_frame_id>laser_frame</gz_frame_id>
+        <update_rate>10</update_rate>
+        <ray>
+          <scan>
+            <horizontal>
+              <samples>360</samples>
+              <min_angle>-3.14159</min_angle>
+              <max_angle>3.14159</max_angle>
+            </horizontal>
+          </scan>
+          <range>
+            <min>0.15</min>
+            <max>12.0</max>
+          </range>
+        </ray>
       </sensor>
     </gazebo>
   </xacro:macro>
-  <!-- New macro added -->
-  <xacro:property name="M_PI" value="3.1415926535897931" />
-  <xacro:macro name="rpi_lidar_sensor" params="
-    prefix:=''
-    frame_name:='laser_frame'
-    parent:='base_link'
-    mesh_file:='file://$(find puzzlebot_description)/meshes/sensors/RPLidar.stl'
-    lidar_base_mass:='0.1755'
-    lidar_base_length:='0.08'
-    lidar_base_width:='0.07'
-    lidar_base_height:='0.05'
-    lidar_base_inertia_pos_x:='0.0'
-    lidar_base_inertia_pos_y:='0.0'
-    lidar_base_inertia_pos_z:='0.021'
-    lidar_base_inertia_pos_r:='0.0'
-    lidar_base_inertia_pos_p:='0.0'
-    lidar_base_inertia_pos_w:='0.0'
-    lidar_base_collision_pos_x:='0.0'
-    lidar_base_collision_pos_y:='0.0'
-    lidar_base_collision_pos_z:='0.021'
-    lidar_base_collision_pos_r:='0.0'
-    lidar_base_collision_pos_p:='0.0'
-    lidar_base_collision_pos_w:='0.0'
-    lidar_base_mesh_pos_x:='0.0'
-    lidar_base_mesh_pos_y:='0.0'
-    lidar_base_mesh_pos_z:='0.025'
-    lidar_base_mesh_pos_r:='0.0'
-    lidar_base_mesh_pos_p:='0.0'
-    lidar_base_mesh_pos_w:='0.0'
-    lidar_base_pos_x:='0.0'
-    lidar_base_pos_y:='0.00'
-    lidar_base_pos_z:='0.070'
-    lidar_base_pos_r:='0.0'
-    lidar_base_pos_p:='0.0'
-    lidar_base_pos_w:='0.0'
-    lidar_pos_x:='0.0'
-    lidar_pos_y:='0.00'
-    lidar_pos_z:='0.035'
-    lidar_pos_r:='0.0'
-    lidar_pos_p:='0.0'
-    lidar_pos_w:='0.0'
-    update_rate:='10'
-    ray_count:='360'
-    min_angle:='-3.14159'
-    max_angle:='3.14159'
-    min_range:='0.15'
-    max_range:='12.0'
-    range_resolution:='0.017'
-    topic_name:='scan'
-    always_on:='true'
-    visualize:='false'
-    ">
-    <link name="${prefix}lidar_base_link">
-        <visual>
-            <origin xyz="${lidar_base_mesh_pos_x} ${lidar_base_mesh_pos_y} ${lidar_base_mesh_pos_z}" rpy="${lidar_base_mesh_pos_r} ${lidar_base_mesh_pos_p} ${lidar_base_mesh_pos_w}"/>
-            <geometry>
-                <mesh filename="${mesh_file}"/>
-            </geometry>
-            <material name="grey"/>
-        </visual>
-        <collision>
-            <origin xyz="${lidar_base_collision_pos_x} ${lidar_base_collision_pos_y} ${lidar_base_collision_pos_z}" rpy="${lidar_base_collision_pos_r} ${lidar_base_collision_pos_p} ${lidar_base_collision_pos_w}"/>
-            <geometry>
-                <box size="${lidar_base_length} ${lidar_base_width} ${lidar_base_height}"/>
-            </geometry>
-        </collision>
-        <inertial>
-            <origin xyz="${lidar_base_inertia_pos_x} ${lidar_base_inertia_pos_y} ${lidar_base_inertia_pos_z}" rpy="${lidar_base_inertia_pos_r} ${lidar_base_inertia_pos_p} ${lidar_base_inertia_pos_w}"/>
-            <mass value="${lidar_base_mass}"/>
-            <xacro:box_inertia mass="${lidar_base_mass}" x="${lidar_base_length}" y="${lidar_base_width}" z="${lidar_base_height}" />
-        </inertial>
-    </link>
-    <link name="${prefix}laser_frame">
-        <visual>
-            <origin xyz="0 0 0" rpy="0 0 0"/>
-            <geometry>
-                <box size="0.005 0.005 0.005"/> <!-- Box shape for lidar -->
-            </geometry>
-            <material name="grey"/>
-        </visual>
-        <collision>
-            <origin xyz="0 0 0" rpy="0 0 0"/>
-            <geometry>
-                <box size="0.005 0.005 0.005"/>
-            </geometry>
-        </collision>
-        <inertial>
-            <origin xyz="0 0 0" rpy="0 0 0"/>
-            <mass value="1e-5"/>
-            <xacro:box_inertia mass="1e-5" x="0.005" y="0.005" z="0.005" />
-        </inertial>
-    </link>
-    <joint name="${prefix}lidar_base_joint" type="fixed">
-        <parent link="${prefix}${parent}"/>
-        <child link="${prefix}lidar_base_link"/>
-        <origin xyz="${lidar_base_pos_x} ${lidar_base_pos_y} ${lidar_base_pos_z}" rpy="${lidar_base_pos_r} ${lidar_base_pos_p} ${lidar_base_pos_w}"/>
-    </joint>
-    <joint name="${prefix}lidar_joint" type="fixed">
-        <parent link="${prefix}lidar_base_link"/>
-        <child link="${prefix}laser_frame"/>
-        <origin xyz="${lidar_pos_x} ${lidar_pos_y} ${lidar_pos_z}" rpy="${lidar_pos_r} ${lidar_pos_p} ${lidar_pos_w}"/>
-    </joint>
-    <gazebo reference="${prefix}laser_frame">
-        <sensor name="${prefix}lidar_sensor" type="gpu_lidar">
-            <topic>${prefix}${topic_name}</topic>
-            <gz_frame_id>${prefix}laser_frame</gz_frame_id>
-            <pose> 0 0 0 0 0 0 </pose>
-            <update_rate>${update_rate}</update_rate>
-            <always_on>${always_on}</always_on>
-            <visualize>${visualize}</visualize>
-            <ray>
-            <scan>
-                <horizontal>
-                <samples>${ray_count}</samples>
-                <resolution>1</resolution>
-                <min_angle>${min_angle}</min_angle>
-                <max_angle>${max_angle}</max_angle>
-                </horizontal>
-                <vertical>
-                <samples>1</samples>
-                <resolution>0.01</resolution>
-                <min_angle>0</min_angle>
-                <max_angle>0</max_angle>
-                </vertical>
-            </scan>
-            <range>
-                <min>${min_range}</min>
-                <max>${max_range}</max>
-                <resolution>${range_resolution}</resolution>
-            </range>
-            </ray>
-        </sensor>
-    </gazebo>
-  </xacro:macro>
 </robot>
