Commit message: Refactor Puzzlebot URDF and Xacro files for improved structure and performance
- Removed unnecessary dependency on xacro in package.xml.
- Updated macros in macros.xacro for inertial calculations and added cylindrical tube inertial macro.
- Enhanced puzzlebot.urdf.xacro by including control and sensor definitions, and restructured wheel and base link definitions.
- Consolidated sensor definitions in sensors.xacro, introducing new parameters for LiDAR configuration and improved inertial properties.
- Created sensors_properties.xacro to centralize sensor-related properties for better maintainability.
- Deleted obsolete robot_base.xacro and wheels.xacro files to streamline the URDF structure.
- Adjusted joint definitions and parameters for wheels and caster to ensure accurate simulation behavior in Gazebo.

File: puzzlebot_nv_ws/src/puzzlebot_ros2/puzzlebot_description/urdf/macros.xacro (robot description, xacro)
@@ -2,41 +2,26 @@
 <robot xmlns:xacro="http://www.ros.org/wiki/xacro">
   <xacro:macro name="box_inertial" params="mass x y z">
-    <inertial>
-      <mass value="${mass}" />
-      <origin xyz="0 0 0" rpy="0 0 0" />
       <inertia
-        ixx="${mass * (y * y + z * z) / 12.0}"
-        ixy="0.0"
-        ixz="0.0"
-        iyy="${mass * (x * x + z * z) / 12.0}"
-        iyz="0.0"
-        izz="${mass * (x * x + y * y) / 12.0}" />
-    </inertial>
+        ixx="${mass/12.0 * (y * y + z * z)}" ixy="0.0" ixz="0.0"
+        iyy="${mass/12.0 * (x * x + z * z)}" iyz="0.0"
+        izz="${mass/12.0 * (x * x + y * y)}" />
   </xacro:macro>
-  <xacro:macro name="cylinder_inertial" params="mass radius length">
-    <inertial>
-      <mass value="${mass}" />
-      <origin xyz="0 0 0" rpy="0 0 0" />
+  <xacro:macro name="cylinder_inertial" params="radius height mass">
       <inertia
-        ixx="${mass * (3.0 * radius * radius + length * length) / 12.0}"
-        ixy="0.0"
-        ixz="0.0"
-        iyy="${mass * (3.0 * radius * radius + length * length) / 12.0}"
-        iyz="0.0"
-        izz="${0.5 * mass * radius * radius}" />
-    </inertial>
+        ixx="${(mass/12.0) * (3.0 * (radius * radius) + height * height)}" ixy="0.0" ixz="0.0"
+        iyy="${(mass/12.0) * (3.0 * (radius * radius) + height * height)}" iyz="0.0"
+        izz="${(mass/2.0) * (radius * radius)}" />
   </xacro:macro>
   <xacro:macro name="sphere_inertial" params="mass radius">
-    <inertial>
-      <mass value="${mass}" />
-      <origin xyz="0 0 0" rpy="0 0 0" />
       <inertia
-        ixx="${0.4 * mass * radius * radius}"
-        ixy="0.0"
-        ixz="0.0"
-        iyy="${0.4 * mass * radius * radius}"
-        iyz="0.0"
+        ixx="${0.4 * mass * radius * radius}" ixy="0.0" ixz="0.0"
+        iyy="${0.4 * mass * radius * radius}" iyz="0.0"
         izz="${0.4 * mass * radius * radius}" />
-    </inertial>
+  </xacro:macro>
+  <xacro:macro name="cylindrical_tube_inertial" params="r1 r2 height mass">
+      <inertia
+        ixx="${(mass/12.0) * (3.0 * (r1 * r1 + r2 * r2) + height * height)}" ixy="0.0" ixz="0.0"
+        iyy="${(mass/12.0) * (3.0 * (r1 * r1 + r2 * r2) + height * height)}" iyz="0.0"
+        izz="${(mass/2.0) * (r1 * r1 + r2 * r2)}" />
   </xacro:macro>
 </robot>

File: puzzlebot_nv_ws/src/puzzlebot_ros2/puzzlebot_description/urdf/puzzlebot.urdf.xacro (robot description, xacro)
@@ -2,15 +2,130 @@
 <robot name="puzzlebot" xmlns:xacro="http://www.ros.org/wiki/xacro">
   <xacro:include filename="$(find puzzlebot_description)/urdf/macros.xacro" />
-  <xacro:include filename="$(find puzzlebot_description)/urdf/robot_base.xacro" />
-  <xacro:include filename="$(find puzzlebot_description)/urdf/wheels.xacro" />
+  <xacro:include filename="$(find puzzlebot_description)/urdf/puzzlebot_control.xacro" />
   <xacro:include filename="$(find puzzlebot_description)/urdf/sensors.xacro" />
+  <xacro:arg name="prefix" default="" />
+<!-- Define materials -->
+  <material name="red"><color rgba="1.0 0.0 0.0 1.0" /></material>
+  <material name="yellow"><color rgba="1.0 1.0 0.0 1.0" /></material>
   <link name="base_footprint" />
-  <joint name="base_footprint_joint" type="fixed">
+  <!-- Base -->
+  <link name="base_link">
+    <inertial>
+      <mass value="1.0" />
+      <inertia ixx="0.01" ixy="0.0" ixz="0.0" iyy="0.01" iyz="0.0" izz="0.01" />
+    </inertial>
+    <visual>
+      <origin xyz="0 0.052 0" rpy="0 0 0" />
+      <geometry>
+        <mesh filename="file://$(find puzzlebot_description)/meshes/Puzzlebot_Jetson_Lidar_Edition_Base.stl" scale="1 1 1"/>
+      </geometry>
+      <material name="red" />
+    </visual>
+    <collision>
+      <origin xyz="0 0.052 0" rpy="0 0 0" />
+      <geometry>
+        <mesh filename="file://$(find puzzlebot_description)/meshes/Puzzlebot_Jetson_Lidar_Edition_Base.stl" scale="1 1 1"/>
+      </geometry>
+    </collision>
+  </link>
+  <joint name="base_link_joint" type="fixed">
     <parent link="base_footprint" />
     <child link="base_link" />
-    <origin xyz="0 0 0" rpy="0 0 0" />
+    <origin xyz="0.052 0 0.05" />
   </joint>
-  <xacro:robot_base />
-  <xacro:puzzlebot_wheels />
-  <xacro:puzzlebot_sensors />
+  <gazebo reference="base_link">
+    <material>Gazebo/Red</material>
+  </gazebo>
+  <!-- Right Wheel -->
+  <link name="right_wheel_link">
+    <inertial>
+      <mass value="0.1" />
+      <inertia ixx="0.001" ixy="0.0" ixz="0.0" iyy="0.001" iyz="0.0" izz="0.001" />
+    </inertial>
+    <visual>
+      <origin xyz="0 0 0" rpy="-1.5708 0 0" />
+      <geometry>
+        <mesh filename="file://$(find puzzlebot_description)/meshes/Puzzlebot_Wheel.stl" scale="1 1 1"/>
+      </geometry>
+      <material name="red" />
+    </visual>
+    <collision>
+      <origin xyz="0 0 0" rpy="-1.5708 0 0" />
+      <geometry>
+        <mesh filename="file://$(find puzzlebot_description)/meshes/Puzzlebot_Wheel.stl" scale="1 1 1"/>
+      </geometry>
+    </collision>
+  </link>
+  <joint name="right_wheel_joint" type="continuous">
+    <parent link="base_link" />
+    <child link="right_wheel_link" />
+    <origin xyz="0 -0.095 -0.0025"/>
+    <axis xyz="0 1 0" />
+  </joint>
+  <gazebo reference="right_wheel_link">
+    <mu1>0.7</mu1>
+    <mu2>0.7</mu2>
+    <material>Gazebo/Red</material>
+  </gazebo>
+  <!-- Left Wheel -->
+  <link name="left_wheel_link">
+    <inertial>
+      <mass value="0.1" />
+      <inertia ixx="0.001" ixy="0.0" ixz="0.0" iyy="0.001" iyz="0.0" izz="0.001" />
+    </inertial>
+    <visual>
+      <origin xyz="0 0 0" rpy="1.5708 0 0" />
+      <geometry>
+        <mesh filename="file://$(find puzzlebot_description)/meshes/Puzzlebot_Wheel.stl" scale="1 1 1"/>
+      </geometry>
+      <material name="red" />
+    </visual>
+    <collision>
+      <origin xyz="0 0 0" rpy="1.5708 0 0" />
+      <geometry>
+        <mesh filename="file://$(find puzzlebot_description)/meshes/Puzzlebot_Wheel.stl" scale="1 1 1"/>
+      </geometry>
+    </collision>
+  </link>
+  <joint name="left_wheel_joint" type="continuous">
+    <parent link="base_link" />
+    <child link="left_wheel_link" />
+    <origin xyz="0 0.095 -0.0025"/>
+    <axis xyz="0 1 0" />
+  </joint>
+  <gazebo reference="left_wheel_link">
+    <mu1>0.7</mu1>
+    <mu2>0.7</mu2>
+    <material>Gazebo/Red</material>
+  </gazebo>
+  <!-- Caster Wheel -->
+  <link name="caster_link">
+    <inertial>
+      <mass value="0.05" />
+      <inertia ixx="0.0005" ixy="0.0" ixz="0.0" iyy="0.0005" iyz="0.0" izz="0.0005" />
+    </inertial>
+    <visual>
+      <geometry>
+        <mesh filename="file://$(find puzzlebot_description)/meshes/Puzzlebot_Caster_Wheel.stl" scale="1 1 1"/>
+      </geometry>
+      <material name="red" />
+    </visual>
+    <collision>
+      <geometry>
+        <mesh filename="file://$(find puzzlebot_description)/meshes/Puzzlebot_Caster_Wheel.stl" scale="1 1 1"/>
+      </geometry>
+    </collision>
+  </link>
+  <joint name="caster_joint" type="fixed">
+    <parent link="base_link" />
+    <child link="caster_link" />
+    <origin xyz="-0.147 0 -0.043"/>
+  </joint>
+  <gazebo reference="caster_link">
+    <mu1>0.1</mu1>
+    <mu2>0.1</mu2>
+    <material>Gazebo/Yellow</material>
+  </gazebo>
+  <xacro:puzzlebot_control prefix="$(arg prefix)" />
+  <xacro:rplidar_sensor prefix="$(arg prefix)" />
 </robot>

File: puzzlebot_nv_ws/src/puzzlebot_ros2/puzzlebot_description/urdf/puzzlebot.xacro (robot description, xacro)
@@ -4,4 +4,4 @@
     <xacro:include filename="$(find puzzlebot_description)/urdf/puzzlebot.urdf.xacro"/>
     <xacro:include filename="$(find puzzlebot_description)/urdf/puzzlebot_control.xacro"/>
-    <xacro:puzzlebot_control prefix="$(arg prefix)"/> <!-- We define prefix so we can have multiple instances of the robot -->
+    <xacro:puzzlebot_control prefix="$(arg prefix)"/>
 </robot>

File: puzzlebot_nv_ws/src/puzzlebot_ros2/puzzlebot_description/urdf/puzzlebot_control.xacro (robot description, xacro)
@@ -3,22 +3,22 @@
     <xacro:macro name= "puzzlebot_control" params="prefix">
         <gazebo>
-            <plugin filename="gz-sim-sensors-system" name="gz::sim::systems::Sensors">
+            <plugin filename="gz-sim-sensors-system" name="ignition::gazebo::systems::Sensors">
                 <render_engine>ogre2</render_engine>
             </plugin>
-            <plugin filename="gz-sim-diff-drive-system" name="gz::sim::systems::DiffDrive">
+            <plugin filename="gz-sim-diff-drive-system" name="ignition::gazebo::systems::DiffDrive">
                 <left_joint>${prefix}left_wheel_joint</left_joint>
                 <right_joint>${prefix}right_wheel_joint</right_joint>
                 <wheel_separation>0.19</wheel_separation>
-                <wheel_radius>0.05</wheel_radius>
-                <topic>${prefix}cmd_vel</topic>
+                <wheel_radius>0.045</wheel_radius>
+                <topic>$/cmd_vel</topic>
                 <tf_topic>/model/puzzlebot/tf</tf_topic>
-                <odom_topic>${prefix}odom</odom_topic>
+                <odom_topic>$/odom</odom_topic>
                 <frame_id>${prefix}odom</frame_id> <!-- Father frame for odometry -->
                 <child_frame_id>${prefix}base_footprint</child_frame_id> <!-- Child frame for odometry -->
                 <odom_publish_frequency>50</odom_publish_frequency>
-                <max_angular_acceleration>1.8</max_angular_acceleration>
+                <max_angular_acceleration>1.2</max_angular_acceleration>
                 <max_angular_velocity>13.0</max_angular_velocity>
             </plugin>
-            <plugin filename="gz-sim-joint-state-publisher-system" name="gz::sim::systems::JointStatePublisher">
+            <plugin filename="gz-sim-joint-state-publisher-system" name="ignition::gazebo::systems::JointStatePublisher">
                 <topic>${prefix}joint_states</topic>
                 <update_rate>50</update_rate>

File: puzzlebot_nv_ws/src/puzzlebot_ros2/puzzlebot_description/urdf/sensors.xacro (robot description, xacro)
@@ -1,68 +1,142 @@
 <?xml version="1.0"?>
 <robot xmlns:xacro="http://www.ros.org/wiki/xacro">
-  <!--
-    puzzlebot_sensors — LiDAR mount and laser_frame definition.
-    Defines the physical TF chain:
-      base_link -> lidar_base_link -> laser_frame
-    The <gazebo> block below is SIMULATION ONLY — it configures the
-    gpu_lidar sensor plugin for Gazebo. On the real robot this block
-    is ignored; the RPLidar A1 driver (rplidar_ros) publishes /scan
-    directly to the laser_frame defined by the joints above.
-  -->
-  <xacro:macro name="puzzlebot_sensors"
-               params="lidar_x:=0.0 lidar_z:=0.055 lidar_mass:=0.05 mesh_scale:=1">
-    <link name="lidar_base_link" />
-    <joint name="lidar_base_joint" type="fixed">
-      <parent link="base_link" />
-      <child link="lidar_base_link" />
-      <origin xyz="${lidar_x} 0 ${lidar_z}" rpy="0 0 0" />
+  <xacro:property name="M_PI" value="3.1415926535897931" />
+  <xacro:macro name="puzzlebot_sensors" params="
+    prefix:=''
+    frame_name:='laser_frame'
+    parent:='base_link'
+    mesh_file:='file://$(find puzzlebot_description)/meshes/RPLidar.stl'
+    lidar_base_mass:='0.1755'
+    lidar_base_length:='0.08'
+    lidar_base_width:='0.07'
+    lidar_base_height:='0.05'
+    lidar_base_inertia_pos_x:='0.0'
+    lidar_base_inertia_pos_y:='0.0'
+    lidar_base_inertia_pos_z:='0.021'
+    lidar_base_inertia_pos_r:='0.0'
+    lidar_base_inertia_pos_p:='0.0'
+    lidar_base_inertia_pos_w:='0.0'
+    lidar_base_collision_pos_x:='0.0'
+    lidar_base_collision_pos_y:='0.0'
+    lidar_base_collision_pos_z:='0.021'
+    lidar_base_collision_pos_r:='0.0'
+    lidar_base_collision_pos_p:='0.0'
+    lidar_base_collision_pos_w:='0.0'
+    lidar_base_mesh_pos_x:='0.0'
+    lidar_base_mesh_pos_y:='0.0'
+    lidar_base_mesh_pos_z:='0.025'
+    lidar_base_mesh_pos_r:='0.0'
+    lidar_base_mesh_pos_p:='0.0'
+    lidar_base_mesh_pos_w:='0.0'
+    lidar_base_pos_x:='0.0'
+    lidar_base_pos_y:='0.00'
+    lidar_base_pos_z:='0.070'
+    lidar_base_pos_r:='0.0'
+    lidar_base_pos_p:='0.0'
+    lidar_base_pos_w:='0.0'
+    lidar_pos_x:='0.0'
+    lidar_pos_y:='0.00'
+    lidar_pos_z:='0.035'
+    lidar_pos_r:='0.0'
+    lidar_pos_p:='0.0'
+    lidar_pos_w:='0.0'
+    update_rate:='10'
+    ray_count:='360'
+    min_angle:='-3.14159'
+    max_angle:='3.14159'
+    min_range:='0.15'
+    max_range:='12.0'
+    range_resolution:='0.017'
+    topic_name:='scan'
+    always_on:='true'
+    visualize:='false'
+    ">
+    <link name="${prefix}lidar_base_link">
+        <visual>
+            <origin xyz="${lidar_base_mesh_pos_x} ${lidar_base_mesh_pos_y} ${lidar_base_mesh_pos_z}" rpy="${lidar_base_mesh_pos_r} ${lidar_base_mesh_pos_p} ${lidar_base_mesh_pos_w}"/>
+            <geometry>
+                <mesh filename="${mesh_file}"/>
+            </geometry>
+            <material name="grey"/>
+        </visual>
+        <collision>
+            <origin xyz="${lidar_base_collision_pos_x} ${lidar_base_collision_pos_y} ${lidar_base_collision_pos_z}" rpy="${lidar_base_collision_pos_r} ${lidar_base_collision_pos_p} ${lidar_base_collision_pos_w}"/>
+            <geometry>
+                <box size="${lidar_base_length} ${lidar_base_width} ${lidar_base_height}"/>
+            </geometry>
+        </collision>
+        <inertial>
+            <origin xyz="${lidar_base_inertia_pos_x} ${lidar_base_inertia_pos_y} ${lidar_base_inertia_pos_z}" rpy="${lidar_base_inertia_pos_r} ${lidar_base_inertia_pos_p} ${lidar_base_inertia_pos_w}"/>
+            <mass value="${lidar_base_mass}"/>
+            <xacro:box_inertia mass="${lidar_base_mass}" x="${lidar_base_length}" y="${lidar_base_width}" z="${lidar_base_height}" />
+        </inertial>
+    </link>
+    <link name="${prefix}laser_frame">
+        <visual>
+            <origin xyz="0 0 0" rpy="0 0 0"/>
+            <geometry>
+                <box size="0.005 0.005 0.005"/> <!-- Box shape for lidar -->
+            </geometry>
+            <material name="grey"/>
+        </visual>
+        <collision>
+            <origin xyz="0 0 0" rpy="0 0 0"/>
+            <geometry>
+                <box size="0.005 0.005 0.005"/>
+            </geometry>
+        </collision>
+        <inertial>
+            <origin xyz="0 0 0" rpy="0 0 0"/>
+            <mass value="1e-5"/>
+            <xacro:box_inertia mass="1e-5" x="0.005" y="0.005" z="0.005" />
+        </inertial>
+    </link>
+    <joint name="${prefix}lidar_base_joint" type="fixed">
+        <parent link="${prefix}${parent}"/>
+        <child link="${prefix}lidar_base_link"/>
+        <origin xyz="${lidar_base_pos_x} ${lidar_base_pos_y} ${lidar_base_pos_z}" rpy="${lidar_base_pos_r} ${lidar_base_pos_p} ${lidar_base_pos_w}"/>
     </joint>
-    <link name="laser_frame">
-      <visual>
-        <origin xyz="0 0 0.021" rpy="0 0 0" />
-        <geometry>
-          <mesh filename="package://puzzlebot_description/meshes/RPLidar.stl"
-                scale="${mesh_scale} ${mesh_scale} ${mesh_scale}" />
-        </geometry>
-        <material name="white">
-          <color rgba="0.9 0.9 0.9 1.0" />
-        </material>
-      </visual>
-      <collision>
-        <origin xyz="0 0 0.021" rpy="0 0 0" />
-        <geometry>
-          <mesh filename="package://puzzlebot_description/meshes/RPLidar.stl"
-                scale="${mesh_scale} ${mesh_scale} ${mesh_scale}" />
-        </geometry>
-      </collision>
-      <xacro:box_inertial mass="${lidar_mass}" x="0.05" y="0.05" z="0.03" />
-    </link>
-    <joint name="laser_frame_joint" type="fixed">
-      <parent link="lidar_base_link" />
-      <child link="laser_frame" />
-      <origin xyz="0 0 0.021" rpy="0 0 0" />
+    <joint name="${prefix}lidar_joint" type="fixed">
+        <parent link="${prefix}lidar_base_link"/>
+        <child link="${prefix}laser_frame"/>
+        <origin xyz="${lidar_pos_x} ${lidar_pos_y} ${lidar_pos_z}" rpy="${lidar_pos_r} ${lidar_pos_p} ${lidar_pos_w}"/>
     </joint>
-    <!-- SIMULATION ONLY — Gazebo gpu_lidar sensor plugin.
-         Not loaded when robot_state_publisher uses puzzlebot.urdf.xacro directly. -->
-    <gazebo reference="laser_frame">
-      <sensor name="lidar_sensor" type="gpu_lidar">
-        <topic>scan</topic>
-        <gz_frame_id>laser_frame</gz_frame_id>
-        <update_rate>10</update_rate>
-        <ray>
-          <scan>
-            <horizontal>
-              <samples>360</samples>
-              <min_angle>-3.14159</min_angle>
-              <max_angle>3.14159</max_angle>
-            </horizontal>
-          </scan>
-          <range>
-            <min>0.15</min>
-            <max>12.0</max>
-          </range>
-        </ray>
-      </sensor>
+    <gazebo reference='${prefix}lidar_base_joint'>
+    <preserveFixedJoint>true</preserveFixedJoint>
     </gazebo>
-  </xacro:macro>
+    <gazebo reference='${prefix}lidar_joint'>
+    <preserveFixedJoint>true</preserveFixedJoint>
+    </gazebo>
+    <gazebo reference="${prefix}laser_frame">
+        <sensor name="${prefix}lidar_sensor" type="gpu_lidar">
+            <topic>${prefix}${topic_name}</topic>
+            <gz_frame_id>${prefix}laser_frame</gz_frame_id>
+            <pose> 0 0 0 0 0 0 </pose>
+            <update_rate>${update_rate}</update_rate>
+            <always_on>${always_on}</always_on>
+            <visualize>${visualize}</visualize>
+            <ray>
+            <scan>
+                <horizontal>
+                <samples>${ray_count}</samples>
+                <resolution>1</resolution>
+                <min_angle>${min_angle}</min_angle>
+                <max_angle>${max_angle}</max_angle>
+                </horizontal>
+                <vertical>
+                <samples>1</samples>
+                <resolution>0.01</resolution>
+                <min_angle>0</min_angle>
+                <max_angle>0</max_angle>
+                </vertical>
+            </scan>
+            <range>
+                <min>${min_range}</min>
+                <max>${max_range}</max>
+                <resolution>${range_resolution}</resolution>
+            </range>
+            </ray>
+        </sensor>
+    </gazebo >
+    </xacro:macro>
 </robot>
